File: PROJE 1.sch (KiCad schematic (older format))
At the start: 11 parts, among them Q1 BC547, Q2 BC547

Commit message: direnç vertical ile değiştrildi
Parts:
- R4: footprint Resistor_THT:R_Axial_DIN0204_L3.6mm_D1.6mm_P5.08mm_Horizontal -> Resistor_THT:R_Axial_DIN0204_L3.6mm_D1.6mm_P2.54mm_Vertical
Changed lines of the file:
@@
 F 0 "R4" H 7620 2896 50  0000 L CNN
 F 1 "470" H 7620 2805 50  0000 L CNN
-F 2 "Resistor_THT:R_Axial_DIN0204_L3.6mm_D1.6mm_P5.08mm_Horizontal" V 7480 2850 50  0001 C CNN
+F 2 "Resistor_THT:R_Axial_DIN0204_L3.6mm_D1.6mm_P2.54mm_Vertical" V 7480 2850 50  0001 C CNN
 F 3 "~" H 7550 2850 50  0001 C CNN
 	1    7550 2850
